File: Circuit_Boards/wireless_charger/wireless_charger.kicad_pcb (KiCad board)
At the start: 4 copper layers, 65 x 69.5 mm, 117 parts, among them J1 Barrel_Jack_Switch, J2 DNP, Q1 DMG7430LFG, Q2 DMG7430LFG, Q3 DMG7430LFG, Q4 DMG7430LFG, Q5 2N7002, Q6 SIA449DJ, Q7 2N7002, Q8 2N7002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

Commit message: cleaned up a bit and mainly added the LED board to the repo
Parts:
- renumbered Fan_12V1 to Fan1
Other:
- board text added: "+"
- board text added: "-"
- board text removed: "12V"
