File: Circuit_Boards/LED_board_B/LED_board.kicad_sch (KiCad schematic)
At the start: 12 parts, among them J1 Conn_01x03, U1 IS32LT3954

Commit message: removed BOM and gerbers for kicad project, to ensure up to date exports
Parts:
- added M1, M2, M3: Lens_Mount, CustomLibrary:LEDiL_Clip, symbol Custom:Lens_Mount
- R2: value 1K -> 1M; Digikey RMCF0603FG1K00CT-ND -> RMCF0603FG1M00CT-ND
Connections:
- net heatsink: no longer LED1.3 (PAD), LED2.3 (PAD), LED3.3 (PAD)
- new net: LED1.3 (PAD), LED2.3 (PAD), LED3.3 (PAD)
Other:
- note removed: "swithc to 1M"
- moved on the sheet: C2, LED1, LED2, LED3, R1
