File: Circuit_Boards/pi_zero_shield/pi_zero_shield.kicad_sch (KiCad schematic)
At the start: 16 parts, among them J1 T1M-10-F-SV-L, J2 Conn_02x20_Odd_Even, J3 T1M-06-X-DV, J4 Screw_Terminal_01x10, J5 Conn_01x02, J6 Conn_01x03, U1 DRV2605LDGS

Commit message: removed BOM and gerbers for kicad project, to ensure up to date exports
Parts:
- BZ1, C1, C2, J1, J3, R1, R2: Buy Digikey skip -> (none)
- C3: Digikey (none) -> 1276-1181-1-ND
- C4, C5: value DNP -> 10uF; Digikey (none) -> 1276-1181-1-ND
- D1: DigiKey MBR0530T1GOSCT-ND -> (none); Digikey (none) -> MBR0530T1GOSCT-ND
- J2, J4, J5, J6, U1: Buy Digikey Buy -> (none)
Other:
- note added: "Power stanbilize caps"
- note removed: "Power stanbilize caps. Extra pads available"
Changed lines of the file:
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@@
     (effects (font (size 1.27 1.27)) (justify left bottom))
   )
-  (text "Power stanbilize caps. Extra pads available" (at 135.89 22.86 0)
+  (text "Power stanbilize caps" (at 146.05 24.13 0)
     (effects (font (size 1.27 1.27)) (justify left bottom))
   )
@@
       (effects (font (size 1.27 1.27)) hide)
     )
-    (property "Buy Digikey" "Buy" (id 5) (at 154.94 144.78 0)
+    (property "Buy Digikey" "" (id 5) (at 154.94 144.78 0)
       (effects (font (size 1.27 1.27)) hide)
     )
@@
       (effects (font (size 1.27 1.27)) hide)
     )
-    (property "Buy Digikey" "skip" (id 5) (at 109.22 172.72 0)
+    (property "Buy Digikey" "" (id 5) (at 109.22 172.72 0)
       (effects (font (size 1.27 1.27)) hide)
     )
@@
       (effects (font (size 1.27 1.27)) hide)
     )
-    (property "Buy Digikey" "skip" (id 5) (at 80.01 106.68 0)
+    (property "Buy Digikey" "" (id 5) (at 80.01 106.68 0)
       (effects (font (size 1.27 1.27)) hide)
     )
@@
       (effects (font (size 1.27 1.27)) hide)
     )
-    (property "Buy Digikey" "skip" (id 5) (at 30.48 106.68 0)
+    (property "Buy Digikey" "" (id 5) (at 30.48 106.68 0)
       (effects (font (size 1.27 1.27)) hide)
     )
@@
       (effects (font (size 1.27 1.27)) hide)
     )
-    (property "Buy Digikey" "Buy" (id 5) (at 142.24 224.79 0)
+    (property "Buy Digikey" "" (id 5) (at 142.24 224.79 0)
       (effects (font (size 1.27 1.27)) hide)
     )
@@
       (effects (font (size 1.27 1.27)) hide)
     )
-    (property "Buy Digikey" "Buy" (id 5) (at 26.67 22.86 0)
+    (property "Buy Digikey" "" (id 5) (at 26.67 22.86 0)
       (effects (font (size 1.27 1.27)) hide)
     )
@@
     )
     (property "DigiKey" "587-TMK316AB7106ML-TCT-ND" (id 4) (at 144.78 31.75 0)
+      (effects (font (size 1.27 1.27)) hide)
+    )
+    (property "Digikey" "1276-1181-1-ND" (id 5) (at 144.78 31.75 0)
       (effects (font (size 1.27 1.27)) hide)
     )
@@
       (effects (font (size 1.27 1.27)) hide)
     )
-    (property "Buy Digikey" "Buy" (id 5) (at 36.83 156.21 0)
+    (property "Buy Digikey" "" (id 5) (at 36.83 156.21 0)
       (effects (font (size 1.27 1.27)) hide)
     )
@@
       (effects (font (size 1.27 1.27)) hide)
     )
-    (property "DigiKey" "MBR0530T1GOSCT-ND" (id 4) (at 120.65 171.45 90)
+    (property "Digikey" "MBR0530T1GOSCT-ND" (id 4) (at 120.65 171.45 90)
       (effects (font (size 1.27 1.27)) hide)
     )
@@
       (effects (font (size 1.27 1.27)) (justify left))
     )
-    (property "Value" "DNP" (id 1) (at 170.18 33.0199 0)
+    (property "Value" "10uF" (id 1) (at 170.18 33.0199 0)
       (effects (font (size 1.27 1.27)) (justify left))
     )
@@
     )
     (property "DigiKey" "" (id 4) (at 167.005 31.75 0)
+      (effects (font (size 1.27 1.27)) hide)
+    )
+    (property "Digikey" "1276-1181-1-ND" (id 5) (at 167.005 31.75 0)
       (effects (font (size 1.27 1.27)) hide)
     )
@@
       (effects (font (size 1.27 1.27)) hide)
     )
-    (property "Buy Digikey" "skip" (id 5) (at 124.46 116.84 0)
+    (property "Buy Digikey" "" (id 5) (at 124.46 116.84 0)
       (effects (font (size 1.27 1.27)) hide)
     )
@@
       (effects (font (size 1.27 1.27)) hide)
     )
-    (property "Buy Digikey" "skip" (id 5) (at 129.54 116.84 0)
+    (property "Buy Digikey" "" (id 5) (at 129.54 116.84 0)
       (effects (font (size 1.27 1.27)) hide)
     )
@@
       (effects (font (size 1.27 1.27)) (justify left))
     )
-    (property "Value" "DNP" (id 1) (at 158.75 33.0199 0)
+    (property "Value" "10uF" (id 1) (at 158.75 33.0199 0)
       (effects (font (size 1.27 1.27)) (justify left))
     )
@@
     )
     (property "DigiKey" "" (id 4) (at 155.575 31.75 0)
+      (effects (font (size 1.27 1.27)) hide)
+    )
+    (property "Digikey" "1276-1181-1-ND" (id 5) (at 155.575 31.75 0)
       (effects (font (size 1.27 1.27)) hide)
     )
@@
       (effects (font (size 1.27 1.27)) hide)
     )
-    (property "Buy Digikey" "skip" (id 6) (at 88.9 48.26 0)
+    (property "Buy Digikey" "" (id 6) (at 88.9 48.26 0)
       (effects (font (size 1.27 1.27)) hide)
     )
@@
       (effects (font (size 1.27 1.27)) hide)
     )
-    (property "Buy Digikey" "Buy" (id 7) (at 57.15 96.52 0)
+    (property "Buy Digikey" "" (id 7) (at 57.15 96.52 0)
       (effects (font (size 1.27 1.27)) hide)
     )
@@
       (effects (font (size 1.27 1.27)) hide)
     )
-    (property "Buy Digikey" "skip" (id 9) (at 71.12 220.98 0)
+    (property "Buy Digikey" "" (id 9) (at 71.12 220.98 0)
       (effects (font (size 1.27 1.27)) hide)
     )
@@
     )
     (path "/be110d7b-fe7b-44f0-8851-960cc7d67573"
-      (reference "C4") (unit 1) (value "DNP") (footprint "Capacitor_SMD:C_1206_3216Metric_Pad1.33x1.80mm_HandSolder")
+      (reference "C4") (unit 1) (value "10uF") (footprint "Capacitor_SMD:C_1206_3216Metric_Pad1.33x1.80mm_HandSolder")
     )
     (path "/7833bb4e-ef34-4a1f-b94e-daf1b7f90e73"
-      (reference "C5") (unit 1) (value "DNP") (footprint "Capacitor_SMD:C_1206_3216Metric_Pad1.33x1.80mm_HandSolder")
+      (reference "C5") (unit 1) (value "10uF") (footprint "Capacitor_SMD:C_1206_3216Metric_Pad1.33x1.80mm_HandSolder")
     )
     (path "/6606cdf2-50ad-4434-aa8d-b85dd7789602"
